File: can_transceiver.kicad_sch (KiCad schematic)
At the start: 4 parts, among them U3 MCP2542FDxMF, U4 MCP2542FDxMF

Commit message: Update
Parts:
- U3, U4: footprint Package_DFN_QFN:DFN-8-1EP_3x3mm_P0.65mm_EP1.55x2.4mm -> Package_SO:SOIC-8-1EP_3.9x4.9mm_P1.27mm_EP2.29x3mm
Changed lines of the file:
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@@
 			)
 		)
-		(property "Footprint" "Package_DFN_QFN:DFN-8-1EP_3x3mm_P0.65mm_EP1.55x2.4mm"
+		(property "Footprint" "Package_SO:SOIC-8-1EP_3.9x4.9mm_P1.27mm_EP2.29x3mm"
 			(at 87.63 142.24 0)
 			(effects
@@
 			)
 		)
-		(property "Footprint" "Package_DFN_QFN:DFN-8-1EP_3x3mm_P0.65mm_EP1.55x2.4mm"
+		(property "Footprint" "Package_SO:SOIC-8-1EP_3.9x4.9mm_P1.27mm_EP2.29x3mm"
 			(at 87.63 76.2 0)
 			(effects

Commit message: Update
Parts:
- C6, C8: value C -> 0.1uF; Mouser (none) -> 603-C0603ZRY5V9BB104
- U3, U4: Mouser (none) -> 579-MCP2542FD-E/SN
Changed lines of the file:
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@@
 			)
 		)
-		(property "Value" "C"
+		(property "Value" "0.1uF"
 			(at 110.49 114.2999 0)
 			(effects
@@
 		)
 		(property "Description" "Unpolarized capacitor"
+			(at 106.68 113.03 0)
+			(effects
+				(font
+					(size 1.27 1.27)
+				)
+				(hide yes)
+			)
+		)
+		(property "Mouser" "603-C0603ZRY5V9BB104"
 			(at 106.68 113.03 0)
 			(effects
@@
 			)
 		)
-		(property "Value" "C"
+		(property "Value" "0.1uF"
 			(at 110.49 45.7199 0)
 			(effects
@@
 		)
 		(property "Description" "Unpolarized capacitor"
+			(at 106.68 44.45 0)
+			(effects
+				(font
+					(size 1.27 1.27)
+				)
+				(hide yes)
+			)
+		)
+		(property "Mouser" "603-C0603ZRY5V9BB104"
 			(at 106.68 44.45 0)
 			(effects
@@
 			)
 		)
+		(property "Mouser" "579-MCP2542FD-E/SN"
+			(at 87.63 129.54 0)
+			(effects
+				(font
+					(size 1.27 1.27)
+				)
+				(hide yes)
+			)
+		)
 		(pin "4"
 		)
@@
 			(at 87.63 63.5 0)
 			(effects
+				(font
+					(size 1.27 1.27)
+				)
+				(hide yes)
+			)
+		)
+		(property "Mouser" "579-MCP2542FD-E/SN"
+			(at 87.63 63.5 0)
+			(effects
