File: USBCAN-X2.kicad_sch (KiCad schematic)
At the start: 15 parts, among them J3 Conn_01x02_Pin, U1 STM32G491CETx, Y1 Crystal_Small

Commit message: Update
Parts:
- added D3: LED, LED_SMD:LED_0603_1608Metric, symbol Device:LED
- added R7: 330, Resistor_SMD:R_0603_1608Metric, symbol Device:R_US
Connections:
- net GND: now also D3.1 (K)
- net LED_PA2: now reaches U1.10 (PA2)
- net LED_PA2: now also R7.1
- new net: D3.2 (A), R7.2
Changed lines of the file:
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@@
+	)
+	(junction
+		(at 160.02 48.26)
+		(diameter 0)
+		(color 0 0 0 0)
 	)
 	(junction
@@
 	(wire
 		(pts
+			(xy 171.45 17.78) (xy 171.45 26.67)
+		)
+		(stroke
+			(width 0)
+			(type default)
+		)
+	)
+	(wire
+		(pts
 			(xy 97.79 67.31) (xy 97.79 76.2)
 		)
@@
 	(wire
 		(pts
+			(xy 171.45 45.72) (xy 171.45 48.26)
+		)
+		(stroke
+			(width 0)
+			(type default)
+		)
+	)
+	(wire
+		(pts
 			(xy 149.86 34.29) (xy 149.86 38.1)
 		)
@@
 	(wire
 		(pts
+			(xy 171.45 34.29) (xy 171.45 38.1)
+		)
+		(stroke
+			(width 0)
+			(type default)
+		)
+	)
+	(wire
+		(pts
 			(xy 160.02 48.26) (xy 149.86 48.26)
 		)
@@
 	(wire
 		(pts
+			(xy 160.02 48.26) (xy 171.45 48.26)
+		)
+		(stroke
+			(width 0)
+			(type default)
+		)
+	)
+	(wire
+		(pts
 			(xy 100.33 67.31) (xy 100.33 76.2)
 		)
@@
 		(pts
 			(xy 53.34 35.56) (xy 64.77 35.56)
+		)
+		(stroke
+			(width 0)
+			(type default)
+		)
+	)
+	(wire
+		(pts
+			(xy 115.57 88.9) (xy 130.81 88.9)
 		)
 		(stroke
@@
 		)
 	)
+	(label "LED_PA2"
+		(at 171.45 25.4 90)
+		(effects
+			(font
+				(size 1.27 1.27)
+			)
+			(justify left bottom)
+		)
+	)
 	(label "3.3V"
 		(at 43.18 90.17 90)
@@
 	(label "3.3V"
 		(at 105.41 67.31 0)
+		(effects
+			(font
+				(size 1.27 1.27)
+			)
+			(justify left bottom)
+		)
+	)
+	(label "LED_PA2"
+		(at 121.92 88.9 0)
 		(effects
 			(font
@@
 	)
 	(symbol
+		(lib_id "Device:R_US")
+		(at 171.45 30.48 0)
+		(unit 1)
+		(exclude_from_sim no)
+		(in_bom yes)
+		(on_board yes)
+		(dnp no)
+		(fields_autoplaced yes)
+		(property "Reference" "R7"
+			(at 173.99 29.2099 0)
+			(effects
+				(font
+					(size 1.27 1.27)
+				)
+				(justify left)
+			)
+		)
+		(property "Value" "330"
+			(at 173.99 31.7499 0)
+			(effects
+				(font
+					(size 1.27 1.27)
+				)
+				(justify left)
+			)
+		)
+		(property "Footprint" "Resistor_SMD:R_0603_1608Metric"
+			(at 172.466 30.734 90)
+			(effects
+				(font
+					(size 1.27 1.27)
+				)
+				(hide yes)
+			)
+		)
+		(property "Datasheet" "~"
+			(at 171.45 30.48 0)
+			(effects
+				(font
+					(size 1.27 1.27)
+				)
+				(hide yes)
+			)
+		)
+		(property "Description" "Resistor, US symbol"
+			(at 171.45 30.48 0)
+			(effects
+				(font
+					(size 1.27 1.27)
+				)
+				(hide yes)
+			)
+		)
+		(pin "2"
+		)
+		(pin "1"
+		)
+		(instances
+			(project "USBCAN-X2"
+				(path "/545a5907-9f92-4fcd-ad93-c3335194e6e8"
+					(reference "R7")
+					(unit 1)
+				)
+			)
+		)
+	)
+	(symbol
 		(lib_id "power:GND")
 		(at 97.79 165.1 0)
@@
 					(unit 1)
 				)
+			)
+		)
+	)
+	(symbol
+		(lib_id "Device:LED")
+		(at 171.45 41.91 90)
+		(unit 1)
+		(exclude_from_sim no)
+		(in_bom yes)
+		(on_board yes)
+		(dnp no)
+		(fields_autoplaced yes)
+		(property "Reference" "D3"
+			(at 175.26 42.2274 90)
+			(effects
+				(font
+					(size 1.27 1.27)
+				)
+				(justify right)
+			)
+		)
+		(property "Value" "LED"
+			(at 175.26 44.7674 90)
+			(effects
+				(font
+					(size 1.27 1.27)
+				)
+				(justify right)
+			)
+		)
+		(property "Footprint" "LED_SMD:LED_0603_1608Metric"
+			(at 171.45 41.91 0)
+			(effects
+				(font
+					(size 1.27 1.27)
+				)
+				(hide yes)
+			)
+		)
+		(property "Datasheet" "~"
+			(at 171.45 41.91 0)
+			(effects
+				(font
+					(size 1.27 1.27)
+				)
+				(hide yes)
+			)
+		)
+		(property "Description" "Light emitting diode"
+			(at 171.45 41.91 0)
+			(effects
+				(font
+					(size 1.27 1.27)
+				)
+				(hide yes)
+			)
+		)
+		(property "Sim.Pins" "1=K 2=A"
+			(at 171.45 41.91 0)
+			(effects
+				(font
+					(size 1.27 1.27)
+				)
+				(hide yes)
+			)
+		)
+		(pin "1"
+		)
+		(pin "2"
+		)
+		(instances
+			(project "USBCAN-X2"
+				(path "/545a5907-9f92-4fcd-ad93-c3335194e6e8"
+					(reference "D3")
+					(unit 1)
+				)

Commit message: Update
Parts:
- C1, C2, C3, C4: Mouser (none) -> 603-C0603ZRY5V9BB104
- C10, C9: value 0.1uF -> 18pF; Mouser (none) -> 791-RF18N180J500CT
- D1: value LED -> LED Green; Mouser (none) -> 710-150060GS83000
- D2: value LED -> LED Blue; Mouser (none) -> 710-150060BS83000
- D3: value LED -> LED Red; Mouser (none) -> 710-150060RS83000
- R1, R2, R7: Mouser (none) -> 774-73L2R33J
- R3: Mouser (none) -> 603-AC0603JR-7W10KL
- R4: Mouser (none) -> 603-SR0603JR-071KL
- U1: Mouser (none) -> 511-STM32G491CET6
- Y1: value Crystal_Small -> 25MHz; Mouser (none) -> 815-ABM725000MHZ4T
Connections:
- net USB_M renamed USB_N
- no-connect marks 0 -> 25
Other:
- moved on the sheet: D1, D2, D3, R1, R2, R7

Commit message: Added an alternative 4-pin debug header
Parts:
- D1: value LED Green -> LED Red; Mouser 710-150060GS83000 -> 710-150060RS83000
- D2: value LED Blue -> LED Green; Mouser 710-150060BS83000 -> 710-150060GS83000
- D3: value LED Red -> LED Blue; Mouser 710-150060RS83000 -> 710-150060BS83000
- J3: value Conn_01x02_Pin -> BOOT0
Other:
- note removed: "BOOT0"
Changed lines of the file:
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@@
 		(comment 1 "Copyright 2025 Karl Yamashita")
-	)
-	(text "BOOT0"
-		(exclude_from_sim no)
-		(at 48.26 110.744 0)
-		(effects
-			(font
-				(size 1.27 1.27)
-			)
-		)
 	)
 	(text "Place each near VDD of STM32"
@@
 		(on_board yes)
 		(dnp no)
-		(fields_autoplaced yes)
 		(property "Reference" "D1"
-			(at 165.1 117.1574 90)
+			(at 155.194 116.84 90)
 			(effects
 				(font
@@
 			)
 		)
-		(property "Value" "LED Green"
-			(at 165.1 119.6974 90)
+		(property "Value" "LED Red"
+			(at 149.606 120.396 90)
 			(effects
 				(font
@@
 			)
 		)
-		(property "Mouser" "710-150060GS83000"
+		(property "Mouser" "710-150060RS83000"
 			(at 161.29 116.84 90)
 			(effects
@@
 		(on_board yes)
 		(dnp no)
-		(fields_autoplaced yes)
 		(property "Reference" "D2"
-			(at 175.26 117.1574 90)
+			(at 170.434 125.984 90)
 			(effects
 				(font
@@
 			)
 		)
-		(property "Value" "LED Blue"
-			(at 175.26 119.6974 90)
+		(property "Value" "LED Green"
+			(at 170.434 129.032 90)
 			(effects
 				(font
@@
 			)
 		)
-		(property "Mouser" "710-150060BS83000"
+		(property "Mouser" "710-150060GS83000"
 			(at 171.45 116.84 90)
 			(effects
@@
 			)
 		)
-		(property "Value" "Conn_01x02_Pin"
-			(at 31.496 106.426 0)
+		(property "Value" "BOOT0"
+			(at 36.83 106.426 0)
 			(effects
 				(font
@@
 			)
 		)
-		(property "Value" "LED Red"
+		(property "Value" "LED Blue"
 			(at 186.69 119.6974 90)
 			(effects
@@
 			)
 		)
-		(property "Mouser" "710-150060RS83000"
+		(property "Mouser" "710-150060BS83000"
 			(at 182.88 116.84 90)
 			(effects

Commit message: Add pull-up to NRST
Parts:
- added R8: 10K, Resistor_SMD:R_0603_1608Metric, symbol Device:R_US
Connections:
- net 3.3V: now also R8.1
- net at U1.7 (PG10): now also R8.2
- no-connect marks 25 -> 24
Changed lines of the file:
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@@
 		(color 0 0 0 0)
 	)
+	(junction
+		(at 77.47 67.31)
+		(diameter 0)
+		(color 0 0 0 0)
+	)
 	(no_connect
 		(at 115.57 96.52)
@@
 	)
 	(no_connect
-		(at 80.01 88.9)
-	)
-	(no_connect
 		(at 80.01 149.86)
 	)
@@
 	(wire
 		(pts
+			(xy 80.01 88.9) (xy 73.66 88.9)
+		)
+		(stroke
+			(width 0)
+			(type default)
+		)
+	)
+	(wire
+		(pts
 			(xy 182.88 109.22) (xy 182.88 113.03)
 		)
@@
 	(wire
 		(pts
+			(xy 73.66 67.31) (xy 77.47 67.31)
+		)
+		(stroke
+			(width 0)
+			(type default)
+		)
+	)
+	(wire
+		(pts
 			(xy 100.33 157.48) (xy 100.33 161.29)
 		)
@@
 	(wire
 		(pts
+			(xy 43.18 85.09) (xy 43.18 92.71)
+		)
+		(stroke
+			(width 0)
+			(type default)
+		)
+	)
+	(wire
+		(pts
+			(xy 171.45 123.19) (xy 182.88 123.19)
+		)
+		(stroke
+			(width 0)
+			(type default)
+		)
+	)
+	(wire
+		(pts
+			(xy 100.33 67.31) (xy 100.33 76.2)
+		)
+		(stroke
+			(width 0)
+			(type default)
+		)
+	)
+	(wire
+		(pts
+			(xy 115.57 83.82) (xy 161.29 83.82)
+		)
+		(stroke
+			(width 0)
+			(type default)
+		)
+	)
+	(wire
+		(pts
+			(xy 67.31 144.78) (xy 80.01 144.78)
+		)
+		(stroke
+			(width 0)
+			(type default)
+		)
+	)
+	(wire
+		(pts
+			(xy 97.79 157.48) (xy 97.79 161.29)
+		)
+		(stroke
+			(width 0)
+			(type default)
+		)
+	)
+	(wire
+		(pts
+			(xy 161.29 120.65) (xy 161.29 123.19)
+		)
+		(stroke
+			(width 0)
+			(type default)
+		)
+	)
+	(wire
+		(pts
 			(xy 77.47 67.31) (xy 92.71 67.31)
 		)
@@
 	(wire
 		(pts
-			(xy 43.18 85.09) (xy 43.18 92.71)
-		)
-		(stroke
-			(width 0)
-			(type default)
-		)
-	)
-	(wire
-		(pts
-			(xy 171.45 123.19) (xy 182.88 123.19)
-		)
-		(stroke
-			(width 0)
-			(type default)
-		)
-	)
-	(wire
-		(pts
-			(xy 100.33 67.31) (xy 100.33 76.2)
-		)
-		(stroke
-			(width 0)
-			(type default)
-		)
-	)
-	(wire
-		(pts
-			(xy 115.57 83.82) (xy 161.29 83.82)
-		)
-		(stroke
-			(width 0)
-			(type default)
-		)
-	)
-	(wire
-		(pts
-			(xy 67.31 144.78) (xy 80.01 144.78)
-		)
-		(stroke
-			(width 0)
-			(type default)
-		)
-	)
-	(wire
-		(pts
-			(xy 97.79 157.48) (xy 97.79 161.29)
-		)
-		(stroke
-			(width 0)
-			(type default)
-		)
-	)
-	(wire
-		(pts
-			(xy 161.29 120.65) (xy 161.29 123.19)
-		)
-		(stroke
-			(width 0)
-			(type default)
-		)
-	)
-	(wire
-		(pts
 			(xy 64.77 107.95) (xy 64.77 110.49)
 		)
@@
 	(wire
 		(pts
+			(xy 73.66 88.9) (xy 73.66 78.74)
+		)
+		(stroke
+			(width 0)
+			(type default)
+		)
+	)
+	(wire
+		(pts
 			(xy 115.57 88.9) (xy 182.88 88.9)
 		)
@@
 		(pts
 			(xy 171.45 86.36) (xy 171.45 101.6)
+		)
+		(stroke
+			(width 0)
+			(type default)
+		)
+	)
+	(wire
+		(pts
+			(xy 73.66 71.12) (xy 73.66 67.31)
 		)
 		(stroke
@@
 					(unit 1)
 				)
+			)
+		)
+	)
+	(symbol
+		(lib_id "Device:R_US")
+		(at 73.66 74.93 0)
+		(unit 1)
+		(exclude_from_sim no)
+		(in_bom yes)
+		(on_board yes)
+		(dnp no)
+		(property "Reference" "R8"
+			(at 68.834 73.406 0)
+			(effects
+				(font
+					(size 1.27 1.27)
+				)
+				(justify left)
+			)
+		)
+		(property "Value" "10K"
+			(at 68.072 76.2 0)
+			(effects
+				(font
+					(size 1.27 1.27)
+				)
+				(justify left)
+			)
+		)
+		(property "Footprint" "Resistor_SMD:R_0603_1608Metric"
+			(at 74.676 75.184 90)
+			(effects
+				(font
+					(size 1.27 1.27)
+				)
+				(hide yes)
+			)
+		)
+		(property "Datasheet" "~"
+			(at 73.66 74.93 0)
+			(effects
+				(font
+					(size 1.27 1.27)
+				)
+				(hide yes)
+			)
+		)
+		(property "Description" "Resistor, US symbol"
+			(at 73.66 74.93 0)
+			(effects
+				(font
+					(size 1.27 1.27)
+				)
+				(hide yes)
+			)
+		)
+		(property "Mouser" "603-AC0603JR-7W10KL"
+			(at 73.66 74.93 0)
+			(effects
+				(font
+					(size 1.27 1.27)
+				)
+				(hide yes)
+			)
+		)
+		(pin "2"
+		)
+		(pin "1"
+		)
+		(instances
+			(project "USBCAN-X2"
+				(path "/545a5907-9f92-4fcd-ad93-c3335194e6e8"
+					(reference "R8")
+					(unit 1)
+				)

Commit message: Clean some tracks up.
Connections:
- net 3.3V: now also D1.2 (A), D2.2 (A), D3.2 (A)
- net GND: no longer D1.1 (K), D2.1 (K), D3.1 (K)
- net LED_PA0: now also R1.2; no longer R1.1
- net LED_PA1: now also R2.2; no longer R2.1
- net LED_PA2: now also R7.2; no longer R7.1
- new net: D1.1 (K), R1.1
- new net: D2.1 (K), R2.1
- new net: D3.1 (K), R7.1
Other:
- moved on the sheet: D1, D2, D3, R1, R2, R7
